File: Neck Board/Neck Board.kicad_sch (KiCad schematic)
At the start: 151 parts, among them J20 TAC005A, P301 Conn_01x06, P302 JST-PHD-14, P303 JST-PHD-16, P304 JST-PHD-10, P305 Conn_01x01, P306 1-Pin, P307 PCS-626-7, Q301 1K, Q302 1W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

Commit message: Start to add base IVAD board
Parts:
- L302, L303, L304: value L -> 0.27uH ?
- L312: value L -> 155A?
- L318: value L -> 155J?
Connections:
- net GUN-VBB is gone; now on net CRT-12V: U1.8 (VBB)
- net GUN-VCC renamed CRT-78V
Changed lines of the file:
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@@
 		)
 	)
-	(global_label "GUN-VCC"
+	(global_label "CRT-78V"
 		(shape output)
 		(at 226.06 193.04 0)
@@
 		)
 		(property "Intersheetrefs" "${INTERSHEET_REFS}"
-			(at 238.1772 193.04 0)
+			(at 237.6328 193.04 0)
 			(effects
 				(font
@@
 		)
 	)
-	(global_label "GUN-VCC"
+	(global_label "CRT-78V"
 		(shape input)
 		(at 171.45 36.83 180)
@@
 		)
 		(property "Intersheetrefs" "${INTERSHEET_REFS}"
-			(at 159.3328 36.83 0)
+			(at 159.8772 36.83 0)
 			(effects
 				(font
@@
 		)
 	)
-	(global_label "GUN-VBB"
+	(global_label "CRT-12V"
 		(shape input)
 		(at 170.18 40.64 180)
@@
 		)
 		(property "Intersheetrefs" "${INTERSHEET_REFS}"
-			(at 158.0628 40.64 0)
+			(at 158.6072 40.64 0)
 			(effects
 				(font
@@
 			)
 		)
-		(property "Value" "L"
-			(at 270.51 118.11 90)
+		(property "Value" "155A?"
+			(at 273.05 118.11 90)
 			(effects
 				(font
@@
 			)
 		)
-		(property "Value" "L"
+		(property "Value" "155J?"
 			(at 307.34 29.845 90)
 			(effects
@@
 			)
 		)
-		(property "Value" "L"
+		(property "Value" "0.27uH ?"
 			(at 194.31 52.07 90)
 			(effects
@@
 			)
 		)
-		(property "Value" "L"
+		(property "Value" "0.27uH ?"
 			(at 194.31 69.215 90)
 			(effects
@@
 			)
 		)
-		(property "Value" "L"
+		(property "Value" "0.27uH ?"
 			(at 194.31 61.595 90)
 			(effects
